File: usb-c-dip-kit.kicad_pcb (KiCad board)
At the start: 2 copper layers, 13.7 x 19.1 mm, 4 parts, among them CN1 USB2.0_C_12pin, CN2 USB_C_DIP_Socket

Commit message: up
Parts:
- removed REF** (x2): Mount_2Pin, $74th:Mount_2Pin
- CN1: footprint $74th:USB-C-12-Pin-MidMount-ali-v2 -> $74th:USB-C-12-Pin-MidMount-ali-v3
- CN2: footprint $usb-type-c-kit:USB2.0-TYPE-C-NOSILK -> $74th:AE-USB2.0-TYPE-C-5077R-NOSILK
- turned CN2 to -90 degrees
