File: usb-c-dip-kit.kicad_sch (KiCad schematic)
At the start: 2 parts, among them CN1 USB2.0_C_12pin, CN2 USB_C_DIP_Socket

Commit message: up
Parts:
- CN1: footprint $74th:USB-C-12-Pin-MidMount-ali -> $usb-type-c-kit:USB-C-12-Pin-MidMount-ali
Changed lines of the file:
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@@
     (property "Reference" "CN1" (id 0) (at 41.275 22.86 0))
     (property "Value" "USB2.0_C_12pin" (id 1) (at 41.275 25.4 0))
-    (property "Footprint" "$74th:USB-C-12-Pin-MidMount-ali" (id 2) (at 40.64 45.72 0)
+    (property "Footprint" "$usb-type-c-kit:USB-C-12-Pin-MidMount-ali" (id 2) (at 40.64 45.72 0)
       (effects (font (size 1.27 1.27)) hide)
     )
@@
   (symbol_instances
     (path "/f57d4f7e-ce77-4da4-a949-56d311b99eb6"
-      (reference "CN1") (unit 1) (value "USB2.0_C_12pin") (footprint "$74th:USB-C-12-Pin-MidMount-ali")
+      (reference "CN1") (unit 1) (value "USB2.0_C_12pin") (footprint "$usb-type-c-kit:USB-C-12-Pin-MidMount-ali")
     )
     (path "/bb4e2dd6-532f-4512-af3d-f00e05846ae6"

Commit message: v2
Parts:
- CN1: footprint $usb-type-c-kit:USB-C-12-Pin-MidMount-ali -> $74th:USB-C-12-Pin-MidMount-ali-v2
- CN2: footprint $usb-type-c-kit:USB2.0-TYPE-C -> $usb-type-c-kit:USB2.0-TYPE-C-NOSILK
Connections:
- net +5V: now reaches CN1.11 (VBUS_B4/A9), CN1.2 (VBUS_A4/B9), CN2.1 (VBUS)
- net GND: now reaches CN1.1 (GND_A1/B12), CN1.12 (GND_A12/B1), CN2.4 (GND), CN2.7 (GND)
Changed lines of the file:
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@@
   (junction (at 64.77 30.48) (diameter 0) (color 0 0 0 0)
   )
-  (junction (at 82.55 38.1) (diameter 0) (color 0 0 0 0)
+  (junction (at 78.74 45.72) (diameter 0) (color 0 0 0 0)
+  )
+  (junction (at 78.74 38.1) (diameter 0) (color 0 0 0 0)
+  )
+  (junction (at 78.74 30.48) (diameter 0) (color 0 0 0 0)
   )
   (junction (at 64.77 50.8) (diameter 0) (color 0 0 0 0)
@@
     (stroke (width 0) (type default) (color 0 0 0 0))
   )
-  (wire (pts (xy 85.09 45.72) (xy 82.55 45.72))
+  (wire (pts (xy 78.74 45.72) (xy 85.09 45.72))
     (stroke (width 0) (type default) (color 0 0 0 0))
   )
-  (wire (pts (xy 64.77 30.48) (xy 85.09 30.48))
+  (wire (pts (xy 64.77 30.48) (xy 78.74 30.48))
     (stroke (width 0) (type default) (color 0 0 0 0))
   )
@@
   )
   (wire (pts (xy 74.93 48.26) (xy 74.93 43.18))
+    (stroke (width 0) (type default) (color 0 0 0 0))
+  )
+  (wire (pts (xy 78.74 27.94) (xy 78.74 30.48))
     (stroke (width 0) (type default) (color 0 0 0 0))
   )
@@
     (stroke (width 0) (type default) (color 0 0 0 0))
   )
-  (wire (pts (xy 82.55 38.1) (xy 85.09 38.1))
+  (wire (pts (xy 78.74 45.72) (xy 78.74 57.15))
+    (stroke (width 0) (type default) (color 0 0 0 0))
+  )
+  (wire (pts (xy 78.74 38.1) (xy 85.09 38.1))
     (stroke (width 0) (type default) (color 0 0 0 0))
   )
@@
     (stroke (width 0) (type default) (color 0 0 0 0))
   )
+  (wire (pts (xy 78.74 38.1) (xy 78.74 45.72))
+    (stroke (width 0) (type default) (color 0 0 0 0))
+  )
   (wire (pts (xy 69.85 35.56) (xy 85.09 35.56))
     (stroke (width 0) (type default) (color 0 0 0 0))
   )
-  (wire (pts (xy 64.77 38.1) (xy 82.55 38.1))
+  (wire (pts (xy 64.77 38.1) (xy 78.74 38.1))
     (stroke (width 0) (type default) (color 0 0 0 0))
   )
   (wire (pts (xy 60.96 45.72) (xy 72.39 45.72))
-    (stroke (width 0) (type default) (color 0 0 0 0))
-  )
-  (wire (pts (xy 82.55 45.72) (xy 82.55 38.1))
     (stroke (width 0) (type default) (color 0 0 0 0))
   )
@@
     (stroke (width 0) (type default) (color 0 0 0 0))
   )
+  (wire (pts (xy 78.74 30.48) (xy 85.09 30.48))
+    (stroke (width 0) (type default) (color 0 0 0 0))
+  )
   (wire (pts (xy 64.77 58.42) (xy 64.77 55.88))
     (stroke (width 0) (type default) (color 0 0 0 0))
+  )
+  (symbol (lib_id "power:GND") (at 78.74 57.15 0) (unit 1)
+    (in_bom yes) (on_board yes) (fields_autoplaced)
+    (property "Reference" "#PWR0101" (id 0) (at 78.74 63.5 0)
+      (effects (font (size 1.27 1.27)) hide)
+    )
+    (property "Value" "GND" (id 1) (at 78.74 62.23 0))
+    (property "Footprint" "" (id 2) (at 78.74 57.15 0)
+      (effects (font (size 1.27 1.27)) hide)
+    )
+    (property "Datasheet" "" (id 3) (at 78.74 57.15 0)
+      (effects (font (size 1.27 1.27)) hide)
+    )
+    (pin "1")
   )
   (symbol (lib_id "$usb-c-dip-kit:USB_C_DIP_Socket") (at 90.17 38.1 0) (unit 1)
@@
       (effects (font (size 1.27 1.27)) (justify left))
     )
-    (property "Footprint" "$usb-type-c-kit:USB2.0-TYPE-C" (id 2) (at 93.98 35.56 0)
+    (property "Footprint" "$usb-type-c-kit:USB2.0-TYPE-C-NOSILK" (id 2) (at 93.98 35.56 0)
       (effects (font (size 1.27 1.27)) hide)
     )
@@
     (property "Reference" "CN1" (id 0) (at 41.275 22.86 0))
     (property "Value" "USB2.0_C_12pin" (id 1) (at 41.275 25.4 0))
-    (property "Footprint" "$usb-type-c-kit:USB-C-12-Pin-MidMount-ali" (id 2) (at 40.64 45.72 0)
+    (property "Footprint" "$74th:USB-C-12-Pin-MidMount-ali-v2" (id 2) (at 40.64 45.72 0)
       (effects (font (size 1.27 1.27)) hide)
     )
@@
     (pin "9")
   )
+  (symbol (lib_id "power:+5V") (at 78.74 27.94 0) (unit 1)
+    (in_bom yes) (on_board yes) (fields_autoplaced)
+    (property "Reference" "#PWR0102" (id 0) (at 78.74 31.75 0)
+      (effects (font (size 1.27 1.27)) hide)
+    )
+    (property "Value" "+5V" (id 1) (at 78.74 22.86 0))
+    (property "Footprint" "" (id 2) (at 78.74 27.94 0)
+      (effects (font (size 1.27 1.27)) hide)
+    )
+    (property "Datasheet" "" (id 3) (at 78.74 27.94 0)
+      (effects (font (size 1.27 1.27)) hide)
+    )
+    (pin "1")
+  )
   (sheet_instances
     (path "/" (page "1"))
   )
   (symbol_instances
+    (path "/083e1a17-4d2b-41f4-9f1b-ca7db66d10c6"
+      (reference "#PWR0101") (unit 1) (value "GND") (footprint "")
+    )
+    (path "/f78d2d90-68bc-4c20-bfb3-6426e74fa17f"
+      (reference "#PWR0102") (unit 1) (value "+5V") (footprint "")
+    )
     (path "/f57d4f7e-ce77-4da4-a949-56d311b99eb6"
-      (reference "CN1") (unit 1) (value "USB2.0_C_12pin") (footprint "$usb-type-c-kit:USB-C-12-Pin-MidMount-ali")
+      (reference "CN1") (unit 1) (value "USB2.0_C_12pin") (footprint "$74th:USB-C-12-Pin-MidMount-ali-v2")
     )
     (path "/bb4e2dd6-532f-4512-af3d-f00e05846ae6"
-      (reference "CN2") (unit 1) (value "USB_C_DIP_Socket") (footprint "$usb-type-c-kit:USB2.0-TYPE-C")
+      (reference "CN2") (unit 1) (value "USB_C_DIP_Socket") (footprint "$usb-type-c-kit:USB2.0-TYPE-C-NOSILK")
     )
   )

Commit message: up
Parts:
- CN1: footprint $74th:USB-C-12-Pin-MidMount-ali-v2 -> $74th:USB-C-12-Pin-MidMount-ali-v3; symbol $74th:USB2.0_C_12pin -> $74th:USB2.0_C_12pin_v2
- CN2: value USB_C_DIP_Socket -> (none); footprint $usb-type-c-kit:USB2.0-TYPE-C-NOSILK -> (none)
Connections:
- no-connect marks 2 -> 0
Changed lines of the file:
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@@
   (junction (at 64.77 38.1) (diameter 0) (color 0 0 0 0)
-  )
-  (junction (at 64.77 55.88) (diameter 0) (color 0 0 0 0)
   )
   (junction (at 64.77 30.48) (diameter 0) (color 0 0 0 0)
@@
   (junction (at 64.77 50.8) (diameter 0) (color 0 0 0 0)
   )
-  (no_connect (at 60.96 43.18))
-  (no_connect (at 60.96 40.64))
+  (junction (at 64.77 45.72) (diameter 0) (color 0 0 0 0)
+  )
   (wire (pts (xy 60.96 35.56) (xy 64.77 35.56))
     (stroke (width 0) (type default) (color 0 0 0 0))
   )
-  (wire (pts (xy 60.96 48.26) (xy 74.93 48.26))
-    (stroke (width 0) (type default) (color 0 0 0 0))
-  )
-  (wire (pts (xy 69.85 55.88) (xy 69.85 35.56))
+  (wire (pts (xy 69.85 50.8) (xy 69.85 35.56))
     (stroke (width 0) (type default) (color 0 0 0 0))
   )
@@
     (stroke (width 0) (type default) (color 0 0 0 0))
   )
-  (wire (pts (xy 60.96 55.88) (xy 64.77 55.88))
+  (wire (pts (xy 60.96 50.8) (xy 64.77 50.8))
     (stroke (width 0) (type default) (color 0 0 0 0))
   )
@@
     (stroke (width 0) (type default) (color 0 0 0 0))
   )
-  (wire (pts (xy 74.93 43.18) (xy 85.09 43.18))
+  (wire (pts (xy 60.96 43.18) (xy 85.09 43.18))
     (stroke (width 0) (type default) (color 0 0 0 0))
   )
-  (wire (pts (xy 64.77 50.8) (xy 67.31 50.8))
+  (wire (pts (xy 64.77 45.72) (xy 67.31 45.72))
+    (stroke (width 0) (type default) (color 0 0 0 0))
+  )
+  (wire (pts (xy 64.77 50.8) (xy 64.77 53.34))
     (stroke (width 0) (type default) (color 0 0 0 0))
   )
@@
   )
   (wire (pts (xy 67.31 33.02) (xy 85.09 33.02))
-    (stroke (width 0) (type default) (color 0 0 0 0))
-  )
-  (wire (pts (xy 74.93 48.26) (xy 74.93 43.18))
     (stroke (width 0) (type default) (color 0 0 0 0))
   )
@@
     (stroke (width 0) (type default) (color 0 0 0 0))
   )
-  (wire (pts (xy 72.39 40.64) (xy 85.09 40.64))
-    (stroke (width 0) (type default) (color 0 0 0 0))
-  )
-  (wire (pts (xy 72.39 45.72) (xy 72.39 40.64))
-    (stroke (width 0) (type default) (color 0 0 0 0))
-  )
-  (wire (pts (xy 64.77 53.34) (xy 64.77 50.8))
+  (wire (pts (xy 60.96 40.64) (xy 85.09 40.64))
     (stroke (width 0) (type default) (color 0 0 0 0))
   )
@@
     (stroke (width 0) (type default) (color 0 0 0 0))
   )
-  (wire (pts (xy 60.96 58.42) (xy 64.77 58.42))
+  (wire (pts (xy 60.96 53.34) (xy 64.77 53.34))
     (stroke (width 0) (type default) (color 0 0 0 0))
   )
-  (wire (pts (xy 64.77 55.88) (xy 69.85 55.88))
+  (wire (pts (xy 64.77 50.8) (xy 69.85 50.8))
     (stroke (width 0) (type default) (color 0 0 0 0))
   )
-  (wire (pts (xy 67.31 50.8) (xy 67.31 33.02))
+  (wire (pts (xy 67.31 45.72) (xy 67.31 33.02))
     (stroke (width 0) (type default) (color 0 0 0 0))
   )
@@
     (stroke (width 0) (type default) (color 0 0 0 0))
   )
-  (wire (pts (xy 60.96 45.72) (xy 72.39 45.72))
+  (wire (pts (xy 60.96 48.26) (xy 64.77 48.26))
     (stroke (width 0) (type default) (color 0 0 0 0))
   )
-  (wire (pts (xy 60.96 53.34) (xy 64.77 53.34))
-    (stroke (width 0) (type default) (color 0 0 0 0))
-  )
-  (wire (pts (xy 60.96 50.8) (xy 64.77 50.8))
+  (wire (pts (xy 60.96 45.72) (xy 64.77 45.72))
     (stroke (width 0) (type default) (color 0 0 0 0))
   )
@@
     (stroke (width 0) (type default) (color 0 0 0 0))
   )
-  (wire (pts (xy 64.77 58.42) (xy 64.77 55.88))
+  (wire (pts (xy 64.77 45.72) (xy 64.77 48.26))
     (stroke (width 0) (type default) (color 0 0 0 0))
   )
@@
       (effects (font (size 1.27 1.27)) (justify left))
     )
-    (property "Value" "USB_C_DIP_Socket" (id 1) (at 95.25 39.3699 0)
+    (property "Value" "" (id 1) (at 95.25 39.3699 0)
       (effects (font (size 1.27 1.27)) (justify left))
     )
-    (property "Footprint" "$usb-type-c-kit:USB2.0-TYPE-C-NOSILK" (id 2) (at 93.98 35.56 0)
+    (property "Footprint" "" (id 2) (at 93.98 35.56 0)
       (effects (font (size 1.27 1.27)) hide)
     )
@@
     (pin "7")
   )
-  (symbol (lib_id "$74th:USB2.0_C_12pin") (at 45.72 45.72 0) (unit 1)
+  (symbol (lib_id "$74th:USB2.0_C_12pin_v2") (at 45.72 45.72 0) (unit 1)
     (in_bom yes) (on_board yes) (fields_autoplaced)
     (property "Reference" "CN1" (id 0) (at 41.275 22.86 0))
     (property "Value" "USB2.0_C_12pin" (id 1) (at 41.275 25.4 0))
-    (property "Footprint" "$74th:USB-C-12-Pin-MidMount-ali-v2" (id 2) (at 40.64 45.72 0)
+    (property "Footprint" "$74th:USB-C-12-Pin-MidMount-ali-v3" (id 2) (at 43.18 67.31 0)
       (effects (font (size 1.27 1.27)) hide)
     )
@@
     (pin "12")
     (pin "2")
-    (pin "3")
     (pin "4")
     (pin "5")
@@
     (pin "7")
     (pin "8")
-    (pin "9")
   )
   (symbol (lib_id "power:+5V") (at 78.74 27.94 0) (unit 1)
@@
     )
     (path "/f57d4f7e-ce77-4da4-a949-56d311b99eb6"
-      (reference "CN1") (unit 1) (value "USB2.0_C_12pin") (footprint "$74th:USB-C-12-Pin-MidMount-ali-v2")
+      (reference "CN1") (unit 1) (value "USB2.0_C_12pin") (footprint "$74th:USB-C-12-Pin-MidMount-ali-v3")
     )
     (path "/bb4e2dd6-532f-4512-af3d-f00e05846ae6"
-      (reference "CN2") (unit 1) (value "USB_C_DIP_Socket") (footprint "$usb-type-c-kit:USB2.0-TYPE-C-NOSILK")
+      (reference "CN2") (unit 1) (value "USB_C_DIP_Socket") (footprint "$74th:AE-USB2.0-TYPE-C-5077R-NOSILK")
     )
   )
